Commit message: demos

File: test/car.urdf (robot description, URDF)
Before this commit: robot drone, 6 links, 5 joints
Links:
- removed link back_left_prop
- removed link back_right_prop
- removed link body
- removed link front_left_prop
- removed link front_right_prop
- added link back_left_wheel, mass 0; collision cylinder length=0.05 radius=0.08; visual cylinder length=0.05 radius=0.08
- added link back_right_wheel, mass 0; collision cylinder length=0.05 radius=0.08; visual cylinder length=0.05 radius=0.08
- added link base_footprint
- added link front_left_wheel, mass 0; collision cylinder length=0.05 radius=0.08; visual cylinder length=0.05 radius=0.08
- added link front_right_wheel, mass 0; collision cylinder length=0.05 radius=0.08; visual cylinder length=0.05 radius=0.08
- link base_link: mass 1.0 -> 2.0; geometry collision box size=0.4 0.3 0.1; visual box size=0.4 0.3 0.1
Joints:
- removed joint base_to_back_left_prop
- removed joint base_to_back_right_prop
- removed joint base_to_front_left_prop
- removed joint base_to_front_right_prop
- removed joint body_link
- added joint base_footprint_to_base_link: type fixed, parent base_footprint, child base_link, origin xyz=0 0 0.08
- added joint base_link_to_back_left_wheel: type revolute, parent base_link, child back_left_wheel, origin xyz=-0.15 0.15 0, axis 0 1 0
- added joint base_link_to_back_right_wheel: type revolute, parent base_link, child back_right_wheel, origin xyz=-0.15 -0.15 0, axis 0 1 0
- added joint base_link_to_front_left_wheel: type revolute, parent base_link, child front_left_wheel, origin xyz=0.15 0.15 0, axis 0 1 0
- added joint base_link_to_front_right_wheel: type revolute, parent base_link, child front_right_wheel, origin xyz=0.15 -0.15 0, axis 0 1 0

Commit message: demos

File: test/car.urdf (robot description, URDF)
Before this commit: robot car, 6 links, 5 joints
Links:
- link back_left_wheel: geometry collision cylinder length=0.07 radius=0.1; visual cylinder length=0.07 radius=0.1
- link back_right_wheel: geometry collision cylinder length=0.07 radius=0.1; visual cylinder length=0.07 radius=0.1
- link front_left_wheel: geometry collision cylinder length=0.07 radius=0.1; visual cylinder length=0.07 radius=0.1
- link front_right_wheel: geometry collision cylinder length=0.07 radius=0.1; visual cylinder length=0.07 radius=0.1
Joints:
- joint base_footprint_to_base_link: origin xyz=0 0 0.08 -> xyz=0 0 0.01
- joint base_link_to_back_left_wheel: axis 0 1 0 -> 0 0 1; origin xyz=-0.15 0.15 0 -> xyz=-0.15 0.185 0 rpy=1.57079 0 0
- joint base_link_to_back_right_wheel: axis 0 1 0 -> 0 0 1; origin xyz=-0.15 -0.15 0 -> xyz=-0.15 -0.185 0 rpy=1.57079 0 0
- joint base_link_to_front_left_wheel: axis 0 1 0 -> 0 0 1; origin xyz=0.15 0.15 0 -> xyz=0.15 0.185 0 rpy=1.57079 0 0
- joint base_link_to_front_right_wheel: axis 0 1 0 -> 0 0 1; origin xyz=0.15 -0.15 0 -> xyz=0.15 -0.185 0 rpy=1.57079 0 0
